File: rotel.kicad_pcb (KiCad board)
At the start: 2 copper layers, 70 x 80 mm, 52 parts, among them J1 GND In +, J2 GND Out +, J3 +40 V GND -40 V, Q1 2SA1016K, Q10 2SD1047, Q11 2SB817, Q2 2SA1016K, Q3 2SA1016K, Q4 2SC1941, Q5 2SA1016K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

Commit message: PCB finished.
Parts:
- moved R10 2.51 mm to (114.8, 79.0)
- moved Q2 1.12 mm to (125.2, 103.9)
- moved C5 1.10 mm to (153.9, 66.3)
- moved Q6 0.91 mm to (121.4, 73.4)
- moved R12 0.63 mm to (150.4, 62.0)
- moved Q9 0.50 mm to (158.5, 62.0)
- moved Q4 0.31 mm to (149.4, 88.4)
Routing:
- net Net-(Q4-Pad1): track 19.5 -> 13.4 mm
- net GND: track 206.0 -> 207.6 mm
- net Net-(C8-Pad1): track 148.4 -> 146.7 mm
- net Net-(D2-Pad1): track 13.9 -> 15.2 mm
- net Net-(C5-Pad2): track 223.2 -> 221.9 mm
- net Net-(Q2-Pad1): track 4.19 -> 5.41 mm
- net Net-(Q1-Pad1): track 41.9 -> 40.8 mm
- net Net-(Q6-Pad2): track 43.7 -> 44.6 mm
- net Net-(Q5-Pad3): track 15.7 -> 14.8 mm
- net Net-(Q5-Pad2): track 30.6 -> 29.7 mm
- net Net-(C4-Pad1): track 68.2 -> 67.7 mm
Other:
- board text added: "19. 4. 2020"
- board text added: "B"
- board text added: "C"
- board text added: "E"
- board text added: "J.F.G.D."
- board text added: "R.S.R."
- board text added: "ROTEL RA02 CLONE"
